Commit message: 22.01.2026

File: arm_robot_description/urdf/arm.xacro (robot description, xacro)
@@ -15,5 +15,5 @@
                 <mesh filename="package://arm_robot_description/meshes/2.parca.STL"/>
             </geometry>
-            <origin rpy="1.57 0 3.14" xyz="0 0 0"/>
+            <origin rpy="0 0 1.57" xyz="0 0 0"/>
             <material name="blue"/>
         </visual>
